File: kicad/Thermometer_Schematic.kicad_sch (KiCad schematic)
At the start: 6 parts, among them U1 LCD-HD44780, U2 DS18B20

Commit message: updated
Parts:
- BT1: value Battery_Cell -> 9V
Other:
- moved on the sheet: R1
Changed lines of the file:
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@@
   (junction (at 138.43 106.68) (diameter 0) (color 0 0 0 0)
   )
-  (junction (at 212.09 76.2) (diameter 0) (color 0 0 0 0)
-  )
-  (junction (at 212.09 88.9) (diameter 0) (color 0 0 0 0)
+  (junction (at 215.9 76.2) (diameter 0) (color 0 0 0 0)
+  )
+  (junction (at 215.9 88.9) (diameter 0) (color 0 0 0 0)
   )
   (junction (at 138.43 116.84) (diameter 0) (color 0 0 0 0)
@@
     (stroke (width 0) (type default))
   )
-  (wire (pts (xy 212.09 88.9) (xy 209.55 88.9))
-    (stroke (width 0) (type default))
-  )
   (wire (pts (xy 142.24 109.22) (xy 151.13 109.22))
     (stroke (width 0) (type default))
@@
     (stroke (width 0) (type default))
   )
-  (wire (pts (xy 220.98 88.9) (xy 212.09 88.9))
+  (wire (pts (xy 224.79 88.9) (xy 215.9 88.9))
     (stroke (width 0) (type default))
   )
@@
     (stroke (width 0) (type default))
   )
-  (wire (pts (xy 212.09 76.2) (xy 201.93 76.2))
+  (wire (pts (xy 215.9 76.2) (xy 201.93 76.2))
     (stroke (width 0) (type default))
   )
@@
     (stroke (width 0) (type default))
   )
-  (wire (pts (xy 212.09 76.2) (xy 212.09 80.01))
+  (wire (pts (xy 215.9 76.2) (xy 215.9 80.01))
     (stroke (width 0) (type default))
   )
@@
     (stroke (width 0) (type default))
   )
+  (wire (pts (xy 209.55 88.9) (xy 215.9 88.9))
+    (stroke (width 0) (type default))
+  )
   (wire (pts (xy 138.43 116.84) (xy 151.13 116.84))
     (stroke (width 0) (type default))
@@
     (stroke (width 0) (type default))
   )
-  (wire (pts (xy 212.09 85.09) (xy 212.09 88.9))
+  (wire (pts (xy 215.9 85.09) (xy 215.9 88.9))
     (stroke (width 0) (type default))
   )
@@
     (stroke (width 0) (type default))
   )
-  (wire (pts (xy 212.09 76.2) (xy 220.98 76.2))
+  (wire (pts (xy 215.9 76.2) (xy 224.79 76.2))
     (stroke (width 0) (type default))
   )
@@
     (effects (font (size 1.27 1.27)) (justify left bottom))
   )
-  (label "U1-DB0" (at 220.98 88.9 180) (fields_autoplaced)
+  (label "U1-DB0" (at 224.79 88.9 180) (fields_autoplaced)
     (effects (font (size 1.27 1.27)) (justify right bottom))
   )
@@
     (effects (font (size 1.27 1.27)) (justify right bottom))
   )
-  (label "A1-VIN" (at 220.98 76.2 180) (fields_autoplaced)
+  (label "A1-VIN" (at 224.79 76.2 180) (fields_autoplaced)
     (effects (font (size 1.27 1.27)) (justify right bottom))
   )
@@
       (effects (font (size 1.27 1.27)) (justify left))
     )
-    (property "Value" "Battery_Cell" (at 120.65 73.533 0)
+    (property "Value" "9V" (at 120.65 73.533 0)
       (effects (font (size 1.27 1.27)) (justify left))
     )
@@
     )
   )
-  (symbol (lib_id "Device:R_Small_US") (at 212.09 82.55 0) (mirror y) (unit 1)
-    (in_bom yes) (on_board yes) (dnp no) (fields_autoplaced)
-    (property "Reference" "R1" (at 209.55 81.915 0)
+  (symbol (lib_id "Device:R_Small_US") (at 215.9 82.55 0) (mirror y) (unit 1)
+    (in_bom yes) (on_board yes) (dnp no) (fields_autoplaced)
+    (property "Reference" "R1" (at 213.36 81.915 0)
       (effects (font (size 1.27 1.27)) (justify left))
     )
-    (property "Value" "220" (at 209.55 84.455 0)
+    (property "Value" "220" (at 213.36 84.455 0)
       (effects (font (size 1.27 1.27)) (justify left))
     )
-    (property "Footprint" "" (at 212.09 82.55 0)
-      (effects (font (size 1.27 1.27)) hide)
-    )
-    (property "Datasheet" "~" (at 212.09 82.55 0)
-      (effects (font (size 1.27 1.27)) hide)
-    )
+    (property "Footprint" "" (at 215.9 82.55 0)
+      (effects (font (size 1.27 1.27)) hide)
+    )
+    (property "Datasheet" "~" (at 215.9 82.55 0)
+      (effects (font (size 1.27 1.27)) hide)
+    )
